Commit message: 更改了 rm_description/urdf/camera.urdf 和 rm_description/urdf/demo.urdf

File: rm_description/urdf/camera.urdf (robot description, URDF)
Before this commit: robot camera, 1 links, 0 joints
Links:
- link Camera_base_link: geometry collision mesh filename=/home/wangwei/ros2_ws/src/ros2_rm_robot/rm_description/mesh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; visual mesh filename=/home/wangwei/ros2_ws/src/ros2_rm_robot/rm_description/mesh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

File: rm_description/urdf/demo.urdf (robot description, URDF)
Before this commit: robot rm_65_description, 13 links, 12 joints
Links:
- link Camera_base_link: geometry collision mesh filename=/home/wangwei/ros2_ws/src/ros2_rm_robot/rm_description/mesh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; visual mesh filename=/home/wangwei/ros2_ws/src/ros2_rm_robot/rm_description/mesh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
- link Link1: geometry collision mesh filename=/home/wangwei/ros2_ws/src/ros2_rm_robot/rm_description/mesh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; visual mesh filename=/home/wangwei/ros2_ws/src/ros2_rm_robot/rm_description/mesh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
- link Link2: geometry collision mesh filename=/home/wangwei/ros2_ws/src/ros2_rm_robot/rm_description/mesh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; visual mesh filename=/home/wangwei/ros2_ws/src/ros2_rm_robot/rm_description/mesh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
- link Link3: geometry collision mesh filename=/home/wangwei/ros2_ws/src/ros2_rm_robot/rm_description/mesh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; visual mesh filename=/home/wangwei/ros2_ws/src/ros2_rm_robot/rm_description/mesh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
- link Link4: geometry collision mesh filename=/home/wangwei/ros2_ws/src/ros2_rm_robot/rm_description/mesh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; visual mesh filename=/home/wangwei/ros2_ws/src/ros2_rm_robot/rm_description/mesh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
- link Link5: geometry collision mesh filename=/home/wangwei/ros2_ws/src/ros2_rm_robot/rm_description/mesh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; visual mesh filename=/home/wangwei/ros2_ws/src/ros2_rm_robot/rm_description/mesh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
- link Link6: geometry collision mesh filename=/home/wangwei/ros2_ws/src/ros2_rm_robot/rm_description/mesh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; visual mesh filename=/home/wangwei/ros2_ws/src/ros2_rm_robot/rm_description/mesh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
- link base_link: geometry collision mesh filename=/home/wangwei/ros2_ws/src/ros2_rm_robot/rm_description/mesh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; visual mesh filename=/home/wangwei/ros2_ws/src/ros2_rm_robot/rm_description/mesh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
- link gripper_base_link: geometry collision mesh filename=/home/wangwei/ros2_ws/src/ros2_rm_robot/rm_description/mesh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; visual mesh filename=/home/wangwei/ros2_ws/src/ros2_rm_robot/rm_description/mesh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
- link gripper_finger1_link1: geometry collision mesh filename=/home/wangwei/ros2_ws/src/ros2_rm_robot/rm_description/mesh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; visual mesh filename=/home/wangwei/ros2_ws/src/ros2_rm_robot/rm_description/mesh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
- link gripper_finger1_link2: geometry collision mesh filename=/home/wangwei/ros2_ws/src/ros2_rm_robot/rm_description/mesh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; visual mesh filename=/home/wangwei/ros2_ws/src/ros2_rm_robot/rm_description/mesh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
- link gripper_finger2_link1: geometry collision mesh filename=/home/wangwei/ros2_ws/src/ros2_rm_robot/rm_description/mesh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; visual mesh filename=/home/wangwei/ros2_ws/src/ros2_rm_robot/rm_description/mesh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
- link gripper_finger2_link2: geometry collision mesh filename=/home/wangwei/ros2_ws/src/ros2_rm_robot/rm_description/mesh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; visual mesh filename=/home/wangwei/ros2_ws/src/ros2_rm_robot/rm_description/mesh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

Commit message: 在机械臂末端添加了二指夹，并相对应修改了gazebo功能包和moveit功能包

File: rm_description/urdf/camera.urdf (robot description, URDF)
Before this commit: robot camera, 1 links, 0 joints
Links:
- link Camera_base_link: geometry collision mesh filename=/home/wangwei/URDF/meshes/camera/camera_stander_no_hole.STL; visual mesh filename=/home/wangwei/URDF/meshes/camera/camera_stander_no_hole.STL

File: rm_description/urdf/demo.urdf (robot description, URDF)
Before this commit: robot rm_65_description, 13 links, 12 joints
Links:
- link Camera_base_link: geometry collision mesh filename=package://rm_description/meshes/camera/camera_stander_no_ho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; visual mesh filename=package://rm_description/meshes/camera/camera_stander_no_ho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
- link Link1: geometry collision mesh filename=package://rm_description/meshes/rm_65_arm/link1.STL; visual mesh filename=package://rm_description/meshes/rm_65_arm/link1.STL
- link Link2: geometry collision mesh filename=package://rm_description/meshes/rm_65_arm/link2.STL; visual mesh filename=package://rm_description/meshes/rm_65_arm/link2.STL
- link Link3: geometry collision mesh filename=package://rm_description/meshes/rm_65_arm/link3.STL; visual mesh filename=package://rm_description/meshes/rm_65_arm/link3.STL
- link Link4: geometry collision mesh filename=package://rm_description/meshes/rm_65_arm/link4.STL; visual mesh filename=package://rm_description/meshes/rm_65_arm/link4.STL
- link Link5: geometry collision mesh filename=package://rm_description/meshes/rm_65_arm/link5.STL; visual mesh filename=package://rm_description/meshes/rm_65_arm/link5.STL
- link Link6: geometry collision mesh filename=package://rm_description/meshes/rm_65_arm/link6.STL; visual mesh filename=package://rm_description/meshes/rm_65_arm/link6.STL
- link base_link: geometry collision mesh filename=package://rm_description/meshes/rm_65_arm/base_link.STL; visual mesh filename=package://rm_description/meshes/rm_65_arm/base_link.STL
- link gripper_base_link: geometry collision mesh filename=package://rm_description/meshes/gripper/base_link.STL; visual mesh filename=package://rm_description/meshes/gripper/base_link.STL
- link gripper_finger1_link1: geometry collision mesh filename=package://rm_description/meshes/gripper/Link1.STL; visual mesh filename=package://rm_description/meshes/gripper/Link1.STL
- link gripper_finger1_link2: geometry collision mesh filename=package://rm_description/meshes/gripper/Link11.STL; visual mesh filename=package://rm_description/meshes/gripper/Link11.STL
- link gripper_finger2_link1: geometry collision mesh filename=package://rm_description/meshes/gripper/Link2.STL; visual mesh filename=package://rm_description/meshes/gripper/Link2.STL
- link gripper_finger2_link2: geometry collision mesh filename=package://rm_description/meshes/gripper/Link22.STL; visual mesh filename=package://rm_description/meshes/gripper/Link22.STL

File: rm_description/urdf/rm_65.urdf (robot description, URDF)
Before this commit: robot rm_65_description, 7 links, 6 joints
Links:
- added link Camera_base_link, mass 0.02; collision mesh filename=package://rm_description/meshes/camera/camera_stander_no_ho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; visual mesh filename=package://rm_description/meshes/camera/camera_stander_no_ho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
- added link gripper_base_link, mass 0.105853592307918; collision mesh filename=package://rm_description/meshes/gripper/base_link.STL; visual mesh filename=package://rm_description/meshes/gripper/base_link.STL
- added link gripper_finger1_link1, mass 0.00647716099397792; collision mesh filename=package://rm_description/meshes/gripper/Link1.STL; visual mesh filename=package://rm_description/meshes/gripper/Link1.STL
- added link gripper_finger1_link2, mass 0.0127543420299361; collision mesh filename=package://rm_description/meshes/gripper/Link11.STL; visual mesh filename=package://rm_description/meshes/gripper/Link11.STL
- added link gripper_finger2_link1, mass 0.00647716099397792; collision mesh filename=package://rm_description/meshes/gripper/Link2.STL; visual mesh filename=package://rm_description/meshes/gripper/Link2.STL
- added link gripper_finger2_link2, mass 0.0127543420299362; collision mesh filename=package://rm_description/meshes/gripper/Link22.STL; visual mesh filename=package://rm_description/meshes/gripper/Link22.STL
Joints:
- added joint finger1_link1_finger1_link2: type revolute, parent gripper_finger1_link1, child gripper_finger1_link2, origin xyz=0.042 0 0.003 rpy=5.0393E-16 5.6225E-16 0.30719, axis 0 0 1, limit lower=-1 upper=0 effort=1 velocity=1
- added joint finger2_link1_finger2_link2: type revolute, parent gripper_finger2_link1, child gripper_finger2_link2, origin xyz=0.042 0 0.015 rpy=-3.641E-16 2.4584E-16 2.8344, axis 0 0 1, limit lower=0 upper=1 effort=1 velocity=1
- added joint gripper_base_joint: type fixed, parent Camera_base_link, child gripper_base_link, origin xyz=0.045 0.039 0.051 rpy=-1.5708 -1.5708 0
- added joint gripper_joint1: type revolute, parent gripper_base_link, child gripper_finger1_link1, origin xyz=0.036 -0.04 -0.019 rpy=-3.0158E-16 -7.1586E-16 -0.30719, axis 0 0 1, limit lower=0 upper=1 effort=1 velocity=1
- added joint gripper_joint2: type revolute, parent gripper_base_link, child gripper_finger2_link1, origin xyz=0.036 0.04 -0.019 rpy=-2.6397E-16 3.7199E-16 0.30719, axis 0 0 1, limit lower=-1 upper=0 effort=1 velocity=1
- added joint joint7: type fixed, parent Link6, child Camera_base_link, origin xyz=-0.045 -0.029 0 rpy=0 0 0

File: rm_description/urdf/rm_65_gazebo.urdf (robot description, URDF)
Before this commit: robot rm_65_description, 7 links, 6 joints
Links:
- added link Camera_base_link, mass 0.02; collision mesh filename=file://$(find rm_description)/meshes/camera/camera_stander_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; visual mesh filename=file://$(find rm_description)/meshes/camera/camera_stander_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
- added link gripper_base_link, mass 0.105853592307918; collision mesh filename=file://$(find rm_description)/meshes/gripper/base_link.STL; visual mesh filename=file://$(find rm_description)/meshes/gripper/base_link.STL
- added link gripper_finger1_link1, mass 0.00647716099397792; collision mesh filename=file://$(find rm_description)/meshes/gripper/Link1.STL; visual mesh filename=file://$(find rm_description)/meshes/gripper/Link1.STL
- added link gripper_finger1_link2, mass 0.0127543420299361; collision mesh filename=file://$(find rm_description)/meshes/gripper/Link11.STL; visual mesh filename=file://$(find rm_description)/meshes/gripper/Link11.STL
- added link gripper_finger2_link1, mass 0.00647716099397792; collision mesh filename=file://$(find rm_description)/meshes/gripper/Link2.STL; visual mesh filename=file://$(find rm_description)/meshes/gripper/Link2.STL
- added link gripper_finger2_link2, mass 0.0127543420299362; collision mesh filename=file://$(find rm_description)/meshes/gripper/Link22.STL; visual mesh filename=file://$(find rm_description)/meshes/gripper/Link22.STL
Joints:
- added joint finger1_link1_finger1_link2: type revolute, parent gripper_finger1_link1, child gripper_finger1_link2, origin xyz=0.042 0 0.003 rpy=5.0393E-16 5.6225E-16 0.30719, axis 0 0 1, limit lower=-1 upper=0 effort=1 velocity=1
- added joint finger2_link1_finger2_link2: type revolute, parent gripper_finger2_link1, child gripper_finger2_link2, origin xyz=0.042 0 0.015 rpy=-3.641E-16 2.4584E-16 2.8344, axis 0 0 1, limit lower=0 upper=1 effort=1 velocity=1
- added joint gripper_base_joint: type fixed, parent Camera_base_link, child gripper_base_link, origin xyz=0.045 0.039 0.051 rpy=-1.5708 -1.5708 0
- added joint gripper_joint1: type revolute, parent gripper_base_link, child gripper_finger1_link1, origin xyz=0.036 -0.04 -0.019 rpy=-3.0158E-16 -7.1586E-16 -0.30719, axis 0 0 1, limit lower=0 upper=1 effort=1 velocity=1
- added joint gripper_joint2: type revolute, parent gripper_base_link, child gripper_finger2_link1, origin xyz=0.036 0.04 -0.019 rpy=-2.6397E-16 3.7199E-16 0.30719, axis 0 0 1, limit lower=-1 upper=0 effort=1 velocity=1
- added joint joint7: type fixed, parent Link6, child Camera_base_link, origin xyz=-0.045 -0.029 0 rpy=0 0 0

File: rm_gazebo/config/gazebo_65_description.urdf.xacro (robot description, xacro)
@@ -1,4 +1,6 @@
 <?xml version="1.0"?>
-<robot xmlns:xacro="http://www.ros.org/wiki/xacro" name="arm">
+<robot xmlns:xacro="http://www.ros.org/wiki/xacro" name="rm_65_description">
+    <!-- Import claw_description urdf file -->
+    <xacro:include filename="$(find rm_description)/urdf/rm_65_gazebo.urdf" />
     <!-- Used for fixing robot to Gazebo 'base_link' 将机械手的基座固定在世界坐标上-->
     <link name="world"/>
@@ -6,49 +8,33 @@
         <parent link="world"/>
         <child link="base_link"/>
-        <origin xyz="0 0 0.815" rpy="0 0 0"/>
     </joint>
-    <!-- Import claw_description urdf file -->
-    <xacro:include filename="$(find rm_description)/urdf/rm_65_gazebo.urdf" />
-    <!-- <xacro:include filename="$(find rm_description)/urdf/camera.urdf" /> -->
-    <!-- <xacro:include filename="$(find rm_description)/urdf/gripper.urdf" /> -->
-    <!-- 连接机械臂与相机 -->
-    <!-- <joint name="connect_camera" type="fixed">
-        <origin xyz="-0.045 -0.029 0" rpy="0 0 0" />
-        <parent link="rm_65_gazebo/Link6" />
-        <child link="camera/Camera_base_link" />
-    </joint> -->
-    <!-- 连接机械臂与夹爪 -->
-    <!-- <joint name="connect_gripper" type="fixed">
-       <origin xyz="0.045 0.039 0.051" rpy="-1.5708 -1.5708 0" />
-       <parent link="camera/Camera_base_link" />
-       <child link="gripper/gripper_base_link" />
-    </joint> -->
     <!-- 对一些link进行gazebo的属性设置 -->
-    <gazebo reference="rm_65_gazebo/base_link">
+    <gazebo reference="base_link">
         <self_collide>false</self_collide>
+        <material>Gazebo/Black</material>
         <gravity>false</gravity>
     </gazebo>
-    <gazebo reference="rm_65_gazebo/Link1">
+    <gazebo reference="Link1">
         <material>Gazebo/Purple</material>
         <self_collide>false</self_collide>
-        <gravity>false</gravity>
+        <gravity>true</gravity>
     </gazebo>
-    <gazebo reference="rm_65_gazebo/Link2">
+    <gazebo reference="Link2">
         <material>Gazebo/Red</material>
         <gravity>false</gravity>
     </gazebo>
-    <gazebo reference="rm_65_gazebo/Link3">
+    <gazebo reference="Link3">
         <material>Gazebo/Blue</material>
         <gravity>false</gravity>
     </gazebo>
-    <gazebo reference="rm_65_gazebo/Link4">
+    <gazebo reference="Link4">
         <material>Gazebo/Green</material>
         <gravity>false</gravity>
     </gazebo>
-    <gazebo reference="rm_65_gazebo/Link5">
+    <gazebo reference="Link5">
         <material>Gazebo/Yellow</material>
         <gravity>false</gravity>
     </gazebo>
-    <gazebo reference="rm_65_gazebo/Link6">
+    <gazebo reference="Link6">
         <material>Gazebo/Orange</material>
         <gravity>false</gravity>
@@ -66,5 +52,5 @@
             <command_interface name="position"/>
             <state_interface name="position">
-                <param name="initial_value">0</param>
+                <param name="initial_value">0.0</param>
             </state_interface>
             <state_interface name="velocity"/>
@@ -73,5 +59,5 @@
             <command_interface name="position"/>
             <state_interface name="position">
-                <param name="initial_value">0</param>
+                <param name="initial_value">0.0</param>
             </state_interface>
             <state_interface name="velocity"/>
@@ -80,5 +66,5 @@
             <command_interface name="position"/>
             <state_interface name="position">
-                <param name="initial_value">0</param>
+                <param name="initial_value">0.0</param>
             </state_interface>
             <state_interface name="velocity"/>
@@ -87,5 +73,5 @@
             <command_interface name="position"/>
             <state_interface name="position">
-                <param name="initial_value">0</param>
+                <param name="initial_value">0.0</param>
             </state_interface>
             <state_interface name="velocity"/>
@@ -94,5 +80,5 @@
             <command_interface name="position"/>
             <state_interface name="position">
-                <param name="initial_value">0</param>
+                <param name="initial_value">0.0</param>
             </state_interface>
             <state_interface name="velocity"/>
@@ -101,5 +87,33 @@
             <command_interface name="position"/>
             <state_interface name="position">
-                <param name="initial_value">0</param>
+                <param name="initial_value">0.0</param>
+            </state_interface>
+            <state_interface name="velocity"/>
+        </joint>
+        <joint name="gripper_joint1">
+            <command_interface name="position"/>
+            <state_interface name="position">
+              <param name="initial_value">0.0</param>
+            </state_interface>
+            <state_interface name="velocity"/>
+        </joint>
+        <joint name="finger1_link1_finger1_link2">
+            <command_interface name="position"/>
+            <state_interface name="position">
+              <param name="initial_value">0.0</param>
+            </state_interface>
+            <state_interface name="velocity"/>
+        </joint>
+        <joint name="gripper_joint2">
+            <command_interface name="position"/>
+            <state_interface name="position">
+              <param name="initial_value">0.0</param>
+            </state_interface>
+            <state_interface name="velocity"/>
+        </joint>
+        <joint name="finger2_link1_finger2_link2">
+            <command_interface name="position"/>
+            <state_interface name="position">
+              <param name="initial_value">0.0</param>
             </state_interface>
             <state_interface name="velocity"/>
@@ -109,6 +123,5 @@
     <gazebo>
         <plugin filename="libgazebo_ros2_control.so" name="gazebo_ros2_control">
-            <!-- <parameters>$(find rm_65_config)/config/gazebo_controllers.yaml</parameters> -->
-            <robot_sim_type>gazebo_ros2_control/GazeboSystem</robot_sim_type>
+            <parameters>$(find rm_gazebo)/config/ros2_controllers.yaml</parameters>
             <robot_param>robot_description</robot_param>
             <robot_param_node>robot_state_publisher</robot_param_node>
